File: baseboard.kicad/soft_power.sch (KiCad schematic (older format))
At the start: 11 parts, among them Q1 IRF7309IPBF, SW1 SW_PUSH

Commit message: fixed switched Value/Reference in soft_power schematic (showed in bad BOM references)
Parts:
- C3: renamed from 1µf1; value C -> 1µF
- C4: renamed from 0.1µf1; value C -> 0.1µF
- C5: renamed from 10µf1; value C -> 10µF
- R1: renamed from 10K1; value R -> 10k
- R11: renamed from 1K1; value R -> 1.1k
- R12: renamed from 300K1; value R -> 300k
- R13: renamed from 100K2; value R -> 100k
- R2: renamed from 100K1; value R -> 100k
Changed lines of the file:
@@
 $EndDescr
 $Comp
-L R 10K1
+L R R1
 U 1 1 5638E982
 P 2850 4050
-F 0 "10K1" V 2930 4050 40  0000 C CNN
-F 1 "R" V 2857 4051 40  0000 C CNN
+F 0 "R1" V 2930 4050 40  0000 C CNN
+F 1 "10k" V 2857 4051 40  0000 C CNN
 F 2 "Resistors_SMD:R_0805_HandSoldering" V 2780 4050 30  0001 C CNN
 F 3 "~" H 2850 4050 30  0000 C CNN
@@
 $EndComp
 $Comp
-L R 100K1
+L R R2
 U 1 1 5638E991
 P 3250 3950
-F 0 "100K1" V 3330 3950 40  0000 C CNN
-F 1 "R" V 3257 3951 40  0000 C CNN
+F 0 "R2" V 3330 3950 40  0000 C CNN
+F 1 "100k" V 3257 3951 40  0000 C CNN
 F 2 "Resistors_SMD:R_0805_HandSoldering" V 3180 3950 30  0001 C CNN
 F 3 "~" H 3250 3950 30  0000 C CNN
@@
 $EndComp
 $Comp
-L R 100K2
+L R R13
 U 1 1 5638F5EC
 P 5950 3700
-F 0 "100K2" V 6030 3700 40  0000 C CNN
-F 1 "R" V 5957 3701 40  0000 C CNN
+F 0 "R13" V 6030 3700 40  0000 C CNN
+F 1 "100k" V 5957 3701 40  0000 C CNN
 F 2 "Resistors_SMD:R_0805_HandSoldering" V 5880 3700 30  0001 C CNN
 F 3 "~" H 5950 3700 30  0000 C CNN
@@
 $EndComp
 $Comp
-L R 1K1
+L R R11
 U 1 1 5638F607
 P 4300 5000
-F 0 "1K1" V 4380 5000 40  0000 C CNN
-F 1 "R" V 4307 5001 40  0000 C CNN
+F 0 "R11" V 4380 5000 40  0000 C CNN
+F 1 "1.1k" V 4307 5001 40  0000 C CNN
 F 2 "Resistors_SMD:R_0805_HandSoldering" V 4230 5000 30  0001 C CNN
 F 3 "~" H 4300 5000 30  0000 C CNN
@@
 $EndComp
 $Comp
-L R 300K1
+L R R12
 U 1 1 5638F619
 P 5700 3950
-F 0 "300K1" V 5780 3950 40  0000 C CNN
-F 1 "R" V 5707 3951 40  0000 C CNN
+F 0 "R12" V 5780 3950 40  0000 C CNN
+F 1 "300k" V 5707 3951 40  0000 C CNN
 F 2 "Resistors_SMD:R_0805_HandSoldering" V 5630 3950 30  0001 C CNN
 F 3 "~" H 5700 3950 30  0000 C CNN
@@
 $EndComp
 $Comp
-L C 10µf1
+L C C5
 U 1 1 5638F658
 P 5450 3750
-F 0 "10µf1" H 5250 3650 40  0000 L CNN
-F 1 "C" H 5456 3665 40  0000 L CNN
+F 0 "C5" H 5350 3650 40  0000 L CNN
+F 1 "10µF" H 5200 3750 40  0000 L CNN
 F 2 "Capacitors_SMD:C_0805_HandSoldering" H 5488 3600 30  0001 C CNN
 F 3 "~" H 5450 3750 60  0000 C CNN
@@
 $EndComp
 $Comp
-L C 1µf1
+L C C3
 U 1 1 5638F671
 P 3050 4300
-F 0 "1µf1" H 3050 4400 40  0000 L CNN
-F 1 "C" H 3056 4215 40  0000 L CNN
+F 0 "C3" H 3050 4400 40  0000 L CNN
+F 1 "1µF" H 3056 4215 40  0000 L CNN
 F 2 "Capacitors_SMD:C_0805_HandSoldering" H 3088 4150 30  0001 C CNN
 F 3 "~" H 3050 4300 60  0000 C CNN
@@
 Connection ~ 3250 3200
 $Comp
-L C 0.1µf1
+L C C4
 U 1 1 5638F756
 P 4650 3500
-F 0 "0.1µf1" H 4650 3600 40  0000 L CNN
-F 1 "C" H 4656 3415 40  0000 L CNN
+F 0 "C4" H 4650 3600 40  0000 L CNN
+F 1 "0.1µF" H 4656 3415 40  0000 L CNN
 F 2 "Capacitors_SMD:C_0805_HandSoldering" H 4688 3350 30  0001 C CNN
 F 3 "~" H 4650 3500 60  0000 C CNN
@@
 	5950 3850 5950 4700
 $Comp
-L GND #PWR032
+L GND #PWR32
 U 1 1 5638F69B
 P 1950 4750
-F 0 "#PWR032" H 1950 4750 30  0001 C CNN
+F 0 "#PWR32" H 1950 4750 30  0001 C CNN
 F 1 "GND" H 1950 4680 30  0001 C CNN
 F 2 "" H 1950 4750 60  0000 C CNN
@@
 	1950 4300 2050 4300
 $Comp
-L GND #PWR033
+L GND #PWR33
 U 1 1 5638F96D
 P 4950 4350
-F 0 "#PWR033" H 4950 4350 30  0001 C CNN
+F 0 "#PWR33" H 4950 4350 30  0001 C CNN
 F 1 "GND" H 4950 4280 30  0001 C CNN
 F 2 "" H 4950 4350 60  0000 C CNN
