File: baseboard.kicad/piggrl_zero_baseboard.sch (KiCad schematic (older format))
At the start: 25 parts, among them P1 PowerBoost 500c, P2 I2C, P3 USB_A, P4 Serial, Q3 Q_PMOS_DGS, Q4 MMBT2222, U1 gpio-header_zero, U2 2.2_tft_ili9340

Commit message: added connection from low-bat on the powerboost to the (till now) unused ID_SD pin
since we already used ID_SC for display-pwm, the whole board won't turn into an spec-compliant hat anyway...
Connections:
- net LowBatOut: now also U1.27 (=ID_SD=)
- no-connect marks 7 -> 5
Changed lines of the file:
@@
 LIBS:valves
 LIBS:raspberry_pins
-LIBS:switches
 LIBS:piggrl_zero_baseboard-cache
 EELAYER 25 0
@@
 $EndComp
 Wire Wire Line
-	5050 5850 5250 5850
+	5050 5850 5200 5850
+Wire Wire Line
+	5200 5850 5250 5850
 Wire Wire Line
 	4750 5850 4550 5850
@@
 	5600 2500 5600 2600
 Wire Wire Line
-	5600 2700 6100 2700
-Wire Wire Line
-	1050 4500 1050 6600
+	5600 2700 5650 2700
+Wire Wire Line
+	5650 2700 5850 2700
+Wire Wire Line
+	5850 2700 6100 2700
+Wire Wire Line
+	1050 4500 1050 4800
+Wire Wire Line
+	1050 4800 1050 5100
+Wire Wire Line
+	1050 5100 1050 5400
+Wire Wire Line
+	1050 5400 1050 5700
+Wire Wire Line
+	1050 5700 1050 6000
+Wire Wire Line
+	1050 6000 1050 6300
+Wire Wire Line
+	1050 6300 1050 6600
 Connection ~ 1050 4800
 Connection ~ 1050 5100
@@
 	2400 1400 2950 1400
 Wire Wire Line
-	2400 750  2400 1400
+	2400 750  2400 900
+Wire Wire Line
+	2400 900  2400 1200
+Wire Wire Line
+	2400 1200 2400 1400
 Wire Wire Line
 	2950 1200 2400 1200
@@
 	2950 800  2500 800
 Wire Wire Line
-	2950 1300 2450 1300
+	2950 1300 2900 1300
+Wire Wire Line
+	2900 1300 2500 1300
 Wire Wire Line
 	2200 750  2400 750
@@
 	7950 3850 7950 4050
 Wire Wire Line
-	7750 3850 7950 3850
+	7750 3850 7900 3850
+Wire Wire Line
+	7900 3850 7950 3850
 Wire Wire Line
 	7850 5050 7950 5050
@@
 	7800 4150 7950 4150
 Wire Wire Line
-	7500 4000 7500 4850
+	7500 4000 7500 4150
+Wire Wire Line
+	7500 4150 7500 4850
 Wire Wire Line
 	7500 4850 7950 4850
@@
 Connection ~ 7900 3850
 Wire Wire Line
-	6100 5800 6950 5800
-Wire Wire Line
-	7550 5050 7550 5600
+	6100 5800 6850 5800
+Wire Wire Line
+	6850 5800 6950 5800
+Wire Wire Line
+	7550 5050 7550 5150
+Wire Wire Line
+	7550 5150 7550 5250
+Wire Wire Line
+	7550 5250 7550 5350
+Wire Wire Line
+	7550 5350 7550 5600
 Connection ~ 7550 5350
 Connection ~ 7550 5250
@@
 	3650 2650 3600 2650
 Wire Wire Line
-	3600 2900 4300 2900
+	3600 2900 4200 2900
+Wire Wire Line
+	4200 2900 4300 2900
 Wire Wire Line
 	3600 2900 3600 2950
@@
 	5600 3100 5650 3100
 Wire Wire Line
-	5650 2700 5650 4100
+	5650 2700 5650 3100
+Wire Wire Line
+	5650 3100 5650 3400
+Wire Wire Line
+	5650 3400 5650 3900
+Wire Wire Line
+	5650 3900 5650 4100
 Connection ~ 5650 2700
 Wire Wire Line
@@
 Connection ~ 5650 3900
 Wire Wire Line
-	4200 2900 4200 4400
+	4200 2900 4200 3700
+Wire Wire Line
+	4200 3700 4200 4400
 Wire Wire Line
 	4200 3700 4300 3700
@@
 	1    0    0    -1
 $EndComp
-NoConn ~ 4300 3800
 NoConn ~ 4400 4750
 NoConn ~ 4400 4850
 NoConn ~ 5500 4850
 NoConn ~ 5500 4750
-NoConn ~ 2450 1300
 Wire Wire Line
 	6100 5800 6100 3800
@@
 	5250 5850 5250 5450
 Connection ~ 5200 5850
+Wire Wire Line
+	4300 3800 2900 3800
+Wire Wire Line
+	2900 3800 2900 1300
+Connection ~ 2900 1300
 $EndSCHEMATC

Commit message: fixed switched Value/Reference in soft_power schematic (showed in bad BOM references)
Changed lines of the file:
@@
 $EndComp
 $Comp
-L GND #PWR01
+L GND #PWR12
 U 1 1 56B8EF7A
 P 5200 5850
-F 0 "#PWR01" H 5200 5600 50  0001 C CNN
+F 0 "#PWR12" H 5200 5600 50  0001 C CNN
 F 1 "GND" H 5200 5700 50  0000 C CNN
 F 2 "" H 5200 5850 60  0000 C CNN
@@
 $EndComp
 $Comp
-L +5V #PWR02
+L +5V #PWR11
 U 1 1 56B8EF94
 P 4550 5850
-F 0 "#PWR02" H 4550 5700 50  0001 C CNN
+F 0 "#PWR11" H 4550 5700 50  0001 C CNN
 F 1 "+5V" H 4550 5990 50  0000 C CNN
 F 2 "" H 4550 5850 60  0000 C CNN
@@
 $EndSheet
 $Comp
-L +5V #PWR03
+L +5V #PWR13
 U 1 1 56B9AD25
 P 5850 2600
-F 0 "#PWR03" H 5850 2450 50  0001 C CNN
+F 0 "#PWR13" H 5850 2450 50  0001 C CNN
 F 1 "+5V" H 5850 2740 50  0000 C CNN
 F 2 "" H 5850 2600 60  0000 C CNN
@@
 $EndComp
 $Comp
-L +5V #PWR04
+L +5V #PWR6
 U 1 1 56B9AD5B
 P 2600 1750
-F 0 "#PWR04" H 2600 1600 50  0001 C CNN
+F 0 "#PWR6" H 2600 1600 50  0001 C CNN
 F 1 "+5V" H 2600 1890 50  0000 C CNN
 F 2 "" H 2600 1750 60  0000 C CNN
@@
 $EndComp
 $Comp
-L GND #PWR05
+L GND #PWR14
 U 1 1 56B9AE12
 P 5850 2700
-F 0 "#PWR05" H 5850 2450 50  0001 C CNN
+F 0 "#PWR14" H 5850 2450 50  0001 C CNN
 F 1 "GND" H 5850 2550 50  0000 C CNN
 F 2 "" H 5850 2700 60  0000 C CNN
@@
 $EndComp
 $Comp
-L GND #PWR06
+L GND #PWR1
 U 1 1 56B9D930
 P 800 4500
-F 0 "#PWR06" H 800 4250 50  0001 C CNN
+F 0 "#PWR1" H 800 4250 50  0001 C CNN
 F 1 "GND" H 800 4350 50  0000 C CNN
 F 2 "" H 800 4500 60  0000 C CNN
@@
 $EndComp
 $Comp
-L GND #PWR07
+L GND #PWR4
 U 1 1 56B9E5B2
 P 2200 750
-F 0 "#PWR07" H 2200 500 50  0001 C CNN
+F 0 "#PWR4" H 2200 500 50  0001 C CNN
 F 1 "GND" H 2200 600 50  0000 C CNN
 F 2 "" H 2200 750 60  0000 C CNN
@@
 $EndComp
 $Comp
-L +BATT #PWR08
+L +BATT #PWR8
 U 1 1 56B9E958
 P 3800 800
-F 0 "#PWR08" H 3800 650 50  0001 C CNN
+F 0 "#PWR8" H 3800 650 50  0001 C CNN
 F 1 "+BATT" H 3800 940 50  0000 C CNN
 F 2 "" H 3800 800 60  0000 C CNN
@@
 +5Vout
 $Comp
-L +BATT #PWR09
+L +BATT #PWR2
 U 1 1 56BA0F04
 P 1700 750
-F 0 "#PWR09" H 1700 600 50  0001 C CNN
+F 0 "#PWR2" H 1700 600 50  0001 C CNN
 F 1 "+BATT" H 1700 890 50  0000 C CNN
 F 2 "" H 1700 750 60  0000 C CNN
@@
 $EndComp
 $Comp
-L GND #PWR010
+L GND #PWR3
 U 1 1 56BA157C
 P 1700 1850
-F 0 "#PWR010" H 1700 1600 50  0001 C CNN
+F 0 "#PWR3" H 1700 1600 50  0001 C CNN
 F 1 "GND" H 1700 1700 50  0000 C CNN
 F 2 "" H 1700 1850 60  0000 C CNN
@@
 $EndComp
 $Comp
-L GND #PWR011
+L GND #PWR5
 U 1 1 56BA1EC4
 P 2500 3350
-F 0 "#PWR011" H 2500 3100 50  0001 C CNN
+F 0 "#PWR5" H 2500 3100 50  0001 C CNN
 F 1 "GND" H 2500 3200 50  0000 C CNN
 F 2 "" H 2500 3350 60  0000 C CNN
@@
 $EndComp
 $Comp
-L GND #PWR012
+L GND #PWR19
 U 1 1 56BA8627
 P 7750 3850
-F 0 "#PWR012" H 7750 3600 50  0001 C CNN
+F 0 "#PWR19" H 7750 3600 50  0001 C CNN
 F 1 "GND" H 7750 3700 50  0000 C CNN
 F 2 "" H 7750 3850 60  0000 C CNN
@@
 $EndComp
 $Comp
-L +3.3V #PWR013
+L +3.3V #PWR17
 U 1 1 56BA8DF9
 P 7500 4000
-F 0 "#PWR013" H 7500 3850 50  0001 C CNN
+F 0 "#PWR17" H 7500 3850 50  0001 C CNN
 F 1 "+3.3V" H 7500 4140 50  0000 C CNN
 F 2 "" H 7500 4000 60  0000 C CNN
@@
 PWM_backlight
 $Comp
-L GND #PWR014
+L GND #PWR18
 U 1 1 56BA9B87
 P 7550 6150
-F 0 "#PWR014" H 7550 5900 50  0001 C CNN
+F 0 "#PWR18" H 7550 5900 50  0001 C CNN
 F 1 "GND" H 7550 6000 50  0000 C CNN
 F 2 "" H 7550 6150 60  0000 C CNN
@@
 $EndComp
 $Comp
-L +5V #PWR015
+L +5V #PWR16
 U 1 1 56BA9D9E
 P 7300 4950
-F 0 "#PWR015" H 7300 4800 50  0001 C CNN
+F 0 "#PWR16" H 7300 4800 50  0001 C CNN
 F 1 "+5V" H 7300 5090 50  0000 C CNN
 F 2 "" H 7300 4950 60  0000 C CNN
@@
 $EndComp
 $Comp
-L +3.3V #PWR016
+L +3.3V #PWR15
 U 1 1 56BB8EAC
 P 6850 5300
-F 0 "#PWR016" H 6850 5150 50  0001 C CNN
+F 0 "#PWR15" H 6850 5150 50  0001 C CNN
 F 1 "+3.3V" H 6850 5440 50  0000 C CNN
 F 2 "" H 6850 5300 60  0000 C CNN
@@
 $EndComp
 $Comp
-L +3.3V #PWR017
+L +3.3V #PWR10
 U 1 1 56BCA582
 P 4300 2500
-F 0 "#PWR017" H 4300 2350 50  0001 C CNN
+F 0 "#PWR10" H 4300 2350 50  0001 C CNN
 F 1 "+3.3V" H 4300 2640 50  0000 C CNN
 F 2 "" H 4300 2500 60  0000 C CNN
@@
 $EndComp
 Wire Wire Line
-	5050 5850 5200 5850
-Wire Wire Line
-	5200 5850 5250 5850
+	5050 5850 5250 5850
 Wire Wire Line
 	4750 5850 4550 5850
@@
 	5600 2500 5600 2600
 Wire Wire Line
-	5600 2700 5650 2700
-Wire Wire Line
-	5650 2700 5850 2700
-Wire Wire Line
-	5850 2700 6100 2700
-Wire Wire Line
-	1050 4500 1050 4800
-Wire Wire Line
-	1050 4800 1050 5100
-Wire Wire Line
-	1050 5100 1050 5400
-Wire Wire Line
-	1050 5400 1050 5700
-Wire Wire Line
-	1050 5700 1050 6000
-Wire Wire Line
-	1050 6000 1050 6300
-Wire Wire Line
-	1050 6300 1050 6600
+	5600 2700 6100 2700
+Wire Wire Line
+	1050 4500 1050 6600
 Connection ~ 1050 4800
 Connection ~ 1050 5100
@@
 	2400 1400 2950 1400
 Wire Wire Line
-	2400 750  2400 900
-Wire Wire Line
-	2400 900  2400 1200
-Wire Wire Line
-	2400 1200 2400 1400
+	2400 750  2400 1400
 Wire Wire Line
 	2950 1200 2400 1200
@@
 	2950 800  2500 800
 Wire Wire Line
-	2950 1300 2900 1300
-Wire Wire Line
-	2900 1300 2500 1300
+	2500 1300 2950 1300
 Wire Wire Line
 	2200 750  2400 750
@@
 	7950 3850 7950 4050
 Wire Wire Line
-	7750 3850 7900 3850
-Wire Wire Line
-	7900 3850 7950 3850
+	7750 3850 7950 3850
 Wire Wire Line
 	7850 5050 7950 5050
@@
 	7800 4150 7950 4150
 Wire Wire Line
-	7500 4000 7500 4150
-Wire Wire Line
-	7500 4150 7500 4850
+	7500 4000 7500 4850
 Wire Wire Line
 	7500 4850 7950 4850
@@
 Connection ~ 7900 3850
 Wire Wire Line
-	6100 5800 6850 5800
-Wire Wire Line
-	6850 5800 6950 5800
-Wire Wire Line
-	7550 5050 7550 5150
-Wire Wire Line
-	7550 5150 7550 5250
-Wire Wire Line
-	7550 5250 7550 5350
-Wire Wire Line
-	7550 5350 7550 5600
+	6100 5800 6950 5800
+Wire Wire Line
+	7550 5050 7550 5600
 Connection ~ 7550 5350
 Connection ~ 7550 5250
@@
 	3650 2650 3600 2650
 Wire Wire Line
-	3600 2900 4200 2900
-Wire Wire Line
-	4200 2900 4300 2900
+	3600 2900 4300 2900
 Wire Wire Line
 	3600 2900 3600 2950
@@
 	5600 3100 5650 3100
 Wire Wire Line
-	5650 2700 5650 3100
-Wire Wire Line
-	5650 3100 5650 3400
-Wire Wire Line
-	5650 3400 5650 3900
-Wire Wire Line
-	5650 3900 5650 4100
+	5650 2700 5650 4100
 Connection ~ 5650 2700
 Wire Wire Line
@@
 Connection ~ 5650 3900
 Wire Wire Line
-	4200 2900 4200 3700
-Wire Wire Line
-	4200 3700 4200 4400
+	4200 2900 4200 4400
 Wire Wire Line
 	4200 3700 4300 3700
@@
 Connection ~ 4200 3700
 $Comp
-L GND #PWR018
+L GND #PWR9
 U 1 1 56BE4980
 P 4200 4400
-F 0 "#PWR018" H 4200 4150 50  0001 C CNN
+F 0 "#PWR9" H 4200 4150 50  0001 C CNN
 F 1 "GND" H 4200 4250 50  0000 C CNN
 F 2 "" H 4200 4400 60  0000 C CNN
@@
 	4300 3300 3350 3300
 $Comp
-L +3.3V #PWR019
+L +3.3V #PWR7
 U 1 1 56BE4AF8
 P 3350 3300
-F 0 "#PWR019" H 3350 3150 50  0001 C CNN
+F 0 "#PWR7" H 3350 3150 50  0001 C CNN
 F 1 "+3.3V" H 3350 3440 50  0000 C CNN
 F 2 "" H 3350 3300 60  0000 C CNN

Commit message: fixed wrong transistor pinout on softpower p-mosfet
common pinout is GSD and not DSG!
Parts:
- removed Q3: Q_PMOS_DGS, TO_SOT_Packages_SMD:SOT-23_Handsoldering, symbol Q_PMOS_DGS
- added Q3: Q_PMOS_GSD, TO_SOT_Packages_SMD:SOT-23_Handsoldering, symbol Q_PMOS_GSD
Connections:
- net Enable: now also Q3.3 (D)
- net soft_power_button/Vout: now also Q3.1 (G)
- net at R3.1: now also Q3.2 (S)
Changed lines of the file:
@@
 $EndComp
 $Comp
-L GND #PWR12
+L GND #PWR01
 U 1 1 56B8EF7A
 P 5200 5850
-F 0 "#PWR12" H 5200 5600 50  0001 C CNN
+F 0 "#PWR01" H 5200 5600 50  0001 C CNN
 F 1 "GND" H 5200 5700 50  0000 C CNN
 F 2 "" H 5200 5850 60  0000 C CNN
@@
 $EndComp
 $Comp
-L +5V #PWR11
+L +5V #PWR02
 U 1 1 56B8EF94
 P 4550 5850
-F 0 "#PWR11" H 4550 5700 50  0001 C CNN
+F 0 "#PWR02" H 4550 5700 50  0001 C CNN
 F 1 "+5V" H 4550 5990 50  0000 C CNN
 F 2 "" H 4550 5850 60  0000 C CNN
@@
 $EndSheet
 $Comp
-L +5V #PWR13
+L +5V #PWR03
 U 1 1 56B9AD25
 P 5850 2600
-F 0 "#PWR13" H 5850 2450 50  0001 C CNN
+F 0 "#PWR03" H 5850 2450 50  0001 C CNN
 F 1 "+5V" H 5850 2740 50  0000 C CNN
 F 2 "" H 5850 2600 60  0000 C CNN
@@
 $EndComp
 $Comp
-L +5V #PWR6
+L +5V #PWR04
 U 1 1 56B9AD5B
 P 2600 1750
-F 0 "#PWR6" H 2600 1600 50  0001 C CNN
+F 0 "#PWR04" H 2600 1600 50  0001 C CNN
 F 1 "+5V" H 2600 1890 50  0000 C CNN
 F 2 "" H 2600 1750 60  0000 C CNN
@@
 $EndComp
 $Comp
-L GND #PWR14
+L GND #PWR05
 U 1 1 56B9AE12
 P 5850 2700
-F 0 "#PWR14" H 5850 2450 50  0001 C CNN
+F 0 "#PWR05" H 5850 2450 50  0001 C CNN
 F 1 "GND" H 5850 2550 50  0000 C CNN
 F 2 "" H 5850 2700 60  0000 C CNN
@@
 $EndComp
 $Comp
-L GND #PWR1
+L GND #PWR06
 U 1 1 56B9D930
 P 800 4500
-F 0 "#PWR1" H 800 4250 50  0001 C CNN
+F 0 "#PWR06" H 800 4250 50  0001 C CNN
 F 1 "GND" H 800 4350 50  0000 C CNN
 F 2 "" H 800 4500 60  0000 C CNN
@@
 $EndComp
 $Comp
-L GND #PWR4
+L GND #PWR07
 U 1 1 56B9E5B2
 P 2200 750
-F 0 "#PWR4" H 2200 500 50  0001 C CNN
+F 0 "#PWR07" H 2200 500 50  0001 C CNN
 F 1 "GND" H 2200 600 50  0000 C CNN
 F 2 "" H 2200 750 60  0000 C CNN
@@
 $EndComp
 $Comp
-L +BATT #PWR8
+L +BATT #PWR08
 U 1 1 56B9E958
 P 3800 800
-F 0 "#PWR8" H 3800 650 50  0001 C CNN
+F 0 "#PWR08" H 3800 650 50  0001 C CNN
 F 1 "+BATT" H 3800 940 50  0000 C CNN
 F 2 "" H 3800 800 60  0000 C CNN
@@
 +5Vout
 $Comp
-L +BATT #PWR2
+L +BATT #PWR09
 U 1 1 56BA0F04
 P 1700 750
-F 0 "#PWR2" H 1700 600 50  0001 C CNN
+F 0 "#PWR09" H 1700 600 50  0001 C CNN
 F 1 "+BATT" H 1700 890 50  0000 C CNN
 F 2 "" H 1700 750 60  0000 C CNN
@@
 $EndComp
 $Comp
-L GND #PWR3
+L GND #PWR010
 U 1 1 56BA157C
 P 1700 1850
-F 0 "#PWR3" H 1700 1600 50  0001 C CNN
+F 0 "#PWR010" H 1700 1600 50  0001 C CNN
 F 1 "GND" H 1700 1700 50  0000 C CNN
 F 2 "" H 1700 1850 60  0000 C CNN
@@
 $EndComp
 $Comp
-L GND #PWR5
+L GND #PWR011
 U 1 1 56BA1EC4
 P 2500 3350
-F 0 "#PWR5" H 2500 3100 50  0001 C CNN
+F 0 "#PWR011" H 2500 3100 50  0001 C CNN
 F 1 "GND" H 2500 3200 50  0000 C CNN
 F 2 "" H 2500 3350 60  0000 C CNN
@@
 $EndComp
 $Comp
-L GND #PWR19
+L GND #PWR012
 U 1 1 56BA8627
 P 7750 3850
-F 0 "#PWR19" H 7750 3600 50  0001 C CNN
+F 0 "#PWR012" H 7750 3600 50  0001 C CNN
 F 1 "GND" H 7750 3700 50  0000 C CNN
 F 2 "" H 7750 3850 60  0000 C CNN
@@
 $EndComp
 $Comp
-L +3.3V #PWR17
+L +3.3V #PWR013
 U 1 1 56BA8DF9
 P 7500 4000
-F 0 "#PWR17" H 7500 3850 50  0001 C CNN
+F 0 "#PWR013" H 7500 3850 50  0001 C CNN
 F 1 "+3.3V" H 7500 4140 50  0000 C CNN
 F 2 "" H 7500 4000 60  0000 C CNN
@@
 PWM_backlight
 $Comp
-L GND #PWR18
+L GND #PWR014
 U 1 1 56BA9B87
 P 7550 6150
-F 0 "#PWR18" H 7550 5900 50  0001 C CNN
+F 0 "#PWR014" H 7550 5900 50  0001 C CNN
 F 1 "GND" H 7550 6000 50  0000 C CNN
 F 2 "" H 7550 6150 60  0000 C CNN
@@
 $EndComp
 $Comp
-L +5V #PWR16
+L +5V #PWR015
 U 1 1 56BA9D9E
 P 7300 4950
-F 0 "#PWR16" H 7300 4800 50  0001 C CNN
+F 0 "#PWR015" H 7300 4800 50  0001 C CNN
 F 1 "+5V" H 7300 5090 50  0000 C CNN
 F 2 "" H 7300 4950 60  0000 C CNN
@@
 $EndComp
 $Comp
-L +3.3V #PWR15
+L +3.3V #PWR016
 U 1 1 56BB8EAC
 P 6850 5300
-F 0 "#PWR15" H 6850 5150 50  0001 C CNN
+F 0 "#PWR016" H 6850 5150 50  0001 C CNN
 F 1 "+3.3V" H 6850 5440 50  0000 C CNN
 F 2 "" H 6850 5300 60  0000 C CNN
@@
 $EndComp
 $Comp
-L +3.3V #PWR10
+L +3.3V #PWR017
 U 1 1 56BCA582
 P 4300 2500
-F 0 "#PWR10" H 4300 2350 50  0001 C CNN
+F 0 "#PWR017" H 4300 2350 50  0001 C CNN
 F 1 "+3.3V" H 4300 2640 50  0000 C CNN
 F 2 "" H 4300 2500 60  0000 C CNN
@@
 Wire Wire Line
 	1650 4500 1800 4500
-$Comp
-L Q_PMOS_DGS Q3
-U 1 1 56BD4D88
-P 1600 1350
-F 0 "Q3" H 1900 1400 50  0000 R CNN
-F 1 "Q_PMOS_DGS" H 2250 1300 50  0000 R CNN
-F 2 "TO_SOT_Packages_SMD:SOT-23_Handsoldering" H 1800 1450 29  0001 C CNN
-F 3 "" H 1600 1350 60  0000 C CNN
-F 4 "Infineon Technologies" H 1600 1350 60  0001 C CNN "ManufacturerName"
-F 5 "SN7002NH6327XTSA2" H 1600 1350 60  0001 C CNN "ManufacturerPartNumber"
-	1    1600 1350
-	1    0    0    -1
-$EndComp
 Wire Wire Line
 	1700 1150 1700 1100
@@
 Connection ~ 4200 3700
 $Comp
-L GND #PWR9
+L GND #PWR018
 U 1 1 56BE4980
 P 4200 4400
-F 0 "#PWR9" H 4200 4150 50  0001 C CNN
+F 0 "#PWR018" H 4200 4150 50  0001 C CNN
 F 1 "GND" H 4200 4250 50  0000 C CNN
 F 2 "" H 4200 4400 60  0000 C CNN
@@
 	4300 3300 3350 3300
 $Comp
-L +3.3V #PWR7
+L +3.3V #PWR019
 U 1 1 56BE4AF8
 P 3350 3300
-F 0 "#PWR7" H 3350 3150 50  0001 C CNN
+F 0 "#PWR019" H 3350 3150 50  0001 C CNN
 F 1 "+3.3V" H 3350 3440 50  0000 C CNN
 F 2 "" H 3350 3300 60  0000 C CNN
@@
 	2900 3800 2900 1300
 Connection ~ 2900 1300
+$Comp
+L Q_PMOS_GSD Q3
+U 1 1 56DAE7F2
+P 1600 1350
+F 0 "Q3" H 1900 1400 50  0000 R CNN
+F 1 "Q_PMOS_GSD" H 2250 1300 50  0000 R CNN
+F 2 "TO_SOT_Packages_SMD:SOT-23_Handsoldering" H 1550 1150 50  0001 C CNN
+F 3 "" H 1600 1350 50  0000 C CNN
+F 4 "Infineon Technologies" H 1600 1350 60  0001 C CNN "ManufacturerName"
+F 5 "BSS84P H6433" H 1600 1350 60  0001 C CNN "ManufacturerPartNumber"
+	1    1600 1350
+	1    0    0    -1
+$EndComp
 $EndSCHEMATC

Commit message: added net_name to usb data lines and rerouted them on the pcb
one less via, and usign kicads wonderfull differential-pair routing tool :-)
Connections:
- net USB_D-: now reaches P3.2 (D-), U1.45 (USB_D-)
- net USB_D+: now reaches P3.3 (D+), U1.46 (USB_D+)
Changed lines of the file:
@@
 	1    0    0    -1
 $EndComp
+Text Label 5500 6100 0    60   ~ 0
+USB_D+
+Text Label 4400 5950 0    60   ~ 0
+USB_D-
 $EndSCHEMATC

Commit message: bugfix: backlicht transistor pinout was BCE instead of common BEC
Parts:
- Q4: symbol Q_NPN_BCE -> Q_NPN_BEC
Connections:
- net GND: now also Q4.2 (E); no longer Q4.3 (E)
- net at R10.2, R7.2, R8.2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: now also Q4.3 (C); no longer Q4.2 (C)
Changed lines of the file:
@@
 $EndComp
 $Comp
-L Q_NPN_BCE Q4
+L Q_NPN_BEC Q4
 U 1 1 56BB78D0
 P 7450 5800

Commit message: ditch mosfet as softpower inverter and use same BJT transistor as the one used for the backlight
Parts:
- removed Q3: Q_PMOS_GSD, TO_SOT_Packages_SMD:SOT-23_Handsoldering, symbol Q_PMOS_GSD
- added Q3: MMBT2222, TO_SOT_Packages_SMD:SOT-23_Handsoldering, symbol Q_NPN_BEC
Connections:
- net Enable: now also Q3.3 (C)
- net GND: now also Q3.2 (E); no longer R3.2
- net soft_power_button/Vout: now also R3.2
- net at R3.1: now also Q3.1 (B)
Other:
- moved on the sheet: R3
Changed lines of the file:
@@
 L R R3
 U 1 1 56BA1501
-P 1700 1700
-F 0 "R3" V 1780 1700 50  0000 C CNN
-F 1 "100k" V 1700 1700 50  0000 C CNN
-F 2 "Resistors_SMD:R_0805_HandSoldering" V 1630 1700 30  0001 C CNN
-F 3 "" H 1700 1700 30  0000 C CNN
-F 4 "Panasonic" H 1700 1700 60  0001 C CNN "ManufacturerName"
-F 5 "ERJ-6ENF1003V" H 1700 1700 60  0001 C CNN "ManufacturerPartNumber"
-	1    1700 1700
+P 1400 1700
+F 0 "R3" V 1480 1700 50  0000 C CNN
+F 1 "100k" V 1400 1700 50  0000 C CNN
+F 2 "Resistors_SMD:R_0805_HandSoldering" V 1330 1700 30  0001 C CNN
+F 3 "" H 1400 1700 30  0000 C CNN
+F 4 "Panasonic" H 1400 1700 60  0001 C CNN "ManufacturerName"
+F 5 "ERJ-6ENF1003V" H 1400 1700 60  0001 C CNN "ManufacturerPartNumber"
+	1    1400 1700
 	1    0    0    -1
 $EndComp
@@
 	1700 1150 1700 1100
 Wire Wire Line
-	1400 2100 1400 1350
+	1400 2100 1400 1850
 Text Label 1800 4500 0    60   ~ 0
 btn_1
@@
 	2900 3800 2900 1300
 Connection ~ 2900 1300
-$Comp
-L Q_PMOS_GSD Q3
-U 1 1 56DAE7F2
-P 1600 1350
-F 0 "Q3" H 1900 1400 50  0000 R CNN
-F 1 "Q_PMOS_GSD" H 2250 1300 50  0000 R CNN
-F 2 "TO_SOT_Packages_SMD:SOT-23_Handsoldering" H 1550 1150 50  0001 C CNN
-F 3 "" H 1600 1350 50  0000 C CNN
-F 4 "Infineon Technologies" H 1600 1350 60  0001 C CNN "ManufacturerName"
-F 5 "BSS84P H6433" H 1600 1350 60  0001 C CNN "ManufacturerPartNumber"
-	1    1600 1350
-	1    0    0    -1
-$EndComp
 Text Label 5500 6100 0    60   ~ 0
 USB_D+
 Text Label 4400 5950 0    60   ~ 0
 USB_D-
+$Comp
+L Q_NPN_BEC Q3
+U 1 1 56E20E5D
+P 1600 1350
+F 0 "Q3" H 1900 1400 50  0000 R CNN
+F 1 "MMBT2222" H 2200 1300 50  0000 R CNN
+F 2 "TO_SOT_Packages_SMD:SOT-23_Handsoldering" H 1800 1450 29  0001 C CNN
+F 3 "" H 1600 1350 60  0000 C CNN
+F 4 "ON Semiconductor" H 1600 1350 60  0001 C CNN "ManufacturerName"
+F 5 "MMBT2222ALT1G" H 1600 1350 60  0001 C CNN "ManufacturerPartNumber"
+	1    1600 1350
+	1    0    0    -1
+$EndComp
+Wire Wire Line
+	1700 1850 1700 1550
+Wire Wire Line
+	1400 1550 1400 1350
 $EndSCHEMATC

Commit message: turns out we don't need the transistor (Q3) at all... so remove it, leaving only the 100k pulldown on the powerboosts enable pin
Parts:
- removed Q3: MMBT2222, TO_SOT_Packages_SMD:SOT-23_Handsoldering, symbol Q_NPN_BEC
Connections:
- net soft_power_button/Vout is gone; now on net GND: R3.2
- net Enable: now also R3.1
Other:
- moved on the sheet: R3
Changed lines of the file:
@@
 L R R3
 U 1 1 56BA1501
-P 1400 1700
-F 0 "R3" V 1480 1700 50  0000 C CNN
-F 1 "100k" V 1400 1700 50  0000 C CNN
-F 2 "Resistors_SMD:R_0805_HandSoldering" V 1330 1700 30  0001 C CNN
-F 3 "" H 1400 1700 30  0000 C CNN
-F 4 "Panasonic" H 1400 1700 60  0001 C CNN "ManufacturerName"
-F 5 "ERJ-6ENF1003V" H 1400 1700 60  0001 C CNN "ManufacturerPartNumber"
-	1    1400 1700
+P 1700 1400
+F 0 "R3" V 1780 1400 50  0000 C CNN
+F 1 "100k" V 1700 1400 50  0000 C CNN
+F 2 "Resistors_SMD:R_0805_HandSoldering" V 1630 1400 30  0001 C CNN
+F 3 "" H 1700 1400 30  0000 C CNN
+F 4 "Panasonic" H 1700 1400 60  0001 C CNN "ManufacturerName"
+F 5 "ERJ-6ENF1003V" H 1700 1400 60  0001 C CNN "ManufacturerPartNumber"
+	1    1700 1400
 	1    0    0    -1
 $EndComp
@@
 L GND #PWR010
 U 1 1 56BA157C
-P 1700 1850
-F 0 "#PWR010" H 1700 1600 50  0001 C CNN
-F 1 "GND" H 1700 1700 50  0000 C CNN
-F 2 "" H 1700 1850 60  0000 C CNN
-F 3 "" H 1700 1850 60  0000 C CNN
-	1    1700 1850
+P 1700 1650
+F 0 "#PWR010" H 1700 1400 50  0001 C CNN
+F 1 "GND" H 1700 1500 50  0000 C CNN
+F 2 "" H 1700 1650 60  0000 C CNN
+F 3 "" H 1700 1650 60  0000 C CNN
+	1    1700 1650
 	1    0    0    -1
 $EndComp
@@
 	3800 800  3800 950
 Wire Wire Line
-	1700 1100 2950 1100
+	1400 1100 2950 1100
 Wire Wire Line
 	2950 800  2500 800
@@
 	1700 1000 1700 750
 Wire Wire Line
-	3400 2100 3400 1200
-Wire Wire Line
-	3400 1200 4250 1200
+	3750 1900 3750 1200
+Wire Wire Line
+	3750 1200 4250 1200
 Wire Wire Line
 	2500 3350 2350 3350
@@
 Connection ~ 6850 5800
 Wire Wire Line
-	3400 2100 1400 2100
+	1400 1900 3750 1900
 Connection ~ 5850 2700
 Wire Wire Line
@@
 	1650 4500 1800 4500
 Wire Wire Line
-	1700 1150 1700 1100
-Wire Wire Line
-	1400 2100 1400 1850
+	1700 1250 1700 1100
+Wire Wire Line
+	1400 1100 1400 1900
 Text Label 1800 4500 0    60   ~ 0
 btn_1
@@
 Text Label 4400 5950 0    60   ~ 0
 USB_D-
-$Comp
-L Q_NPN_BEC Q3
-U 1 1 56E20E5D
-P 1600 1350
-F 0 "Q3" H 1900 1400 50  0000 R CNN
-F 1 "MMBT2222" H 2200 1300 50  0000 R CNN
-F 2 "TO_SOT_Packages_SMD:SOT-23_Handsoldering" H 1800 1450 29  0001 C CNN
-F 3 "" H 1600 1350 60  0000 C CNN
-F 4 "ON Semiconductor" H 1600 1350 60  0001 C CNN "ManufacturerName"
-F 5 "MMBT2222ALT1G" H 1600 1350 60  0001 C CNN "ManufacturerPartNumber"
-	1    1600 1350
-	1    0    0    -1
-$EndComp
-Wire Wire Line
-	1700 1850 1700 1550
-Wire Wire Line
-	1400 1550 1400 1350
+Wire Wire Line
+	1700 1650 1700 1550
+Connection ~ 1700 1100
+Text GLabel 3750 1200 0    60   Input ~ 0
+Enable
 $EndSCHEMATC
